File: hardware/kicad/cpu_memory.kicad_sch (KiCad schematic)
At the start: 34 parts, among them U1 Z84C0004 (Z80 CMOS), U10 74HCT04, U11 74HCT74 paging on / AY clock, U2 SST39SF040 flash, pages 0-31, U3 AS6C4008 SRAM, pages 32-63, U4 74HCT670 page bits 0-3, U5 74HCT670 page bits 4-5, U6 74HCT138 I/O 80h-BFh, U7 74HCT138 I/O 00h-7Fh, U8 74HCT32, U9 74HCT32

Commit message: Add the routed 4-layer PCB and move the board to SMD parts
Schematic:
- Z80, TMS9918A, AY-3-8910 and 82C55 stay DIP-40 in sockets (the
  chips in hand), the SST39SF040 flash is a socketed DIP-32 so it can
  be programmed; everything else is surface mount: AS6C4008 SOP-32,
  AS6C62256 SOP-28 VRAM, logic in SOIC, ATmega328P-AU TQFP-32, 0805.
- The UM245R module becomes an FT245RL (SSOP-28) with a USB-C socket
  (GCT USB4105), wired as FTDI's self-powered figure 6.2.
- 74HC670 instead of the 74HCT670, no longer made in SOIC; all its
  inputs come from CMOS outputs.
- MMBT4401 video transistor with SOT-23 pins 1 B, 2 E, 3 C; the TO-92
  pin numbers used before were wrong.
- SCART and PS/2 go to headers for short cables (no KiCad footprints;
  smaller board). DB9s, USB-C and the 12 V jack stay on the board.
- Pin tables checked against the manufacturers' datasheets;
  check_footprints.py confirms every symbol pin has a pad.

PCB (gen_pcb.py, KiCad 9 Python):
- 138 x 105 mm, 4 layers: tracks on F.Cu, In2.Cu and B.Cu, In1.Cu an
  unbroken GND plane, +5V as 0.4 mm tracks plus a fill on In2.Cu.
- Connectors on the top edge, the DIP sockets in one row, each
  group's SMD parts packed beside and below its socket with each
  chip's 100 nF next to it. One-sided SMD assembly.
- Routed with Freerouting 2.5.0. The DSN is adjusted so only GND may
  use In1.Cu and the boundary is inset by the edge clearance.
- KiCad DRC with schematic parity: 0 violations, 0 unconnected pads,
  0 footprint errors. Only silkscreen warnings remain. ERC 0.

Not built or tested.

Co-Authored-By: Claude Opus 5.5 <noreply@anthropic.com>
Parts:
- C10, C11, C12, C13, C14, C15, C16, C6, C7, C8, C9: footprint Capacitor_THT:C_Disc_D5.0mm_W2.5mm_P5.00mm -> Capacitor_SMD:C_0805_2012Metric
- JP1: footprint Connector_PinHeader_2.54mm:PinHeader_1x02_P2.54mm_Vertical -> Jumper:SolderJumper-2_P1.3mm_Open_TrianglePad1.0x1.5mm
- R1, R10, R11, R2, R3, R4, R5, R6, R7, R8, R9: footprint Resistor_THT:R_Axial_DIN0207_L6.3mm_D2.5mm_P10.16mm_Horizontal -> Resistor_SMD:R_0805_2012Metric
- U1: footprint Package_DIP:DIP-40_W15.24mm -> Package_DIP:DIP-40_W15.24mm_Socket
- U10, U11, U8, U9: footprint Package_DIP:DIP-14_W7.62mm -> Package_SO:SOIC-14_3.9x8.7mm_P1.27mm
- U2: footprint Package_DIP:DIP-32_W15.24mm -> Package_DIP:DIP-32_W15.24mm_Socket
- U3: footprint Package_DIP:DIP-32_W15.24mm -> Package_SO:SOP-32_11.305x20.495mm_P1.27mm
- U4, U5: footprint Package_DIP:DIP-16_W7.62mm -> Package_SO:SOIC-16_3.9x9.9mm_P1.27mm; symbol zl80:74HCT670 -> zl80:74HC670
- U6, U7: footprint Package_DIP:DIP-16_W7.62mm -> Package_SO:SOIC-16_3.9x9.9mm_P1.27mm
