File: hardware/kicad/keyboard_usb.kicad_sch (KiCad schematic)
At the start: 17 parts, among them J6 PS/2 keyboard, J7 ISP for the ATmega, J8 Expansion (8255 PA, PC4-7), U21 82C55A, U22 ATmega328P: PS/2 to key matrix, U23 UM245R USB FIFO module, U27 74HCT32 USB FIFO strobes, U28 74HCT125 USB status on D0, D1

Commit message: Add the routed 4-layer PCB and move the board to SMD parts
Schematic:
- Z80, TMS9918A, AY-3-8910 and 82C55 stay DIP-40 in sockets (the
  chips in hand), the SST39SF040 flash is a socketed DIP-32 so it can
  be programmed; everything else is surface mount: AS6C4008 SOP-32,
  AS6C62256 SOP-28 VRAM, logic in SOIC, ATmega328P-AU TQFP-32, 0805.
- The UM245R module becomes an FT245RL (SSOP-28) with a USB-C socket
  (GCT USB4105), wired as FTDI's self-powered figure 6.2.
- 74HC670 instead of the 74HCT670, no longer made in SOIC; all its
  inputs come from CMOS outputs.
- MMBT4401 video transistor with SOT-23 pins 1 B, 2 E, 3 C; the TO-92
  pin numbers used before were wrong.
- SCART and PS/2 go to headers for short cables (no KiCad footprints;
  smaller board). DB9s, USB-C and the 12 V jack stay on the board.
- Pin tables checked against the manufacturers' datasheets;
  check_footprints.py confirms every symbol pin has a pad.

PCB (gen_pcb.py, KiCad 9 Python):
- 138 x 105 mm, 4 layers: tracks on F.Cu, In2.Cu and B.Cu, In1.Cu an
  unbroken GND plane, +5V as 0.4 mm tracks plus a fill on In2.Cu.
- Connectors on the top edge, the DIP sockets in one row, each
  group's SMD parts packed beside and below its socket with each
  chip's 100 nF next to it. One-sided SMD assembly.
- Routed with Freerouting 2.5.0. The DSN is adjusted so only GND may
  use In1.Cu and the boundary is inset by the edge clearance.
- KiCad DRC with schematic parity: 0 violations, 0 unconnected pads,
  0 footprint errors. Only silkscreen warnings remain. ERC 0.

Not built or tested.

Co-Authored-By: Claude Opus 5.5 <noreply@anthropic.com>
Parts:
- added C36: 100n, Capacitor_SMD:C_0805_2012Metric, symbol zl80:C
- added C37: 4.7u, Capacitor_SMD:C_0805_2012Metric, symbol zl80:C
- added C38: 100n (U23), Capacitor_SMD:C_0805_2012Metric, symbol zl80:C
- added C39: 10n, Capacitor_SMD:C_0805_2012Metric, symbol zl80:C
- added J10: USB-C (GCT USB4105-GF-A), Connector_USB:USB_C_Receptacle_GCT_USB4105-xx-A_16P_TopMnt_Horizontal, symbol zl80:USB_C
- added R48: 4.7k, Resistor_SMD:R_0805_2012Metric, symbol zl80:R
- added R49, R50: 10k, Resistor_SMD:R_0805_2012Metric, symbol zl80:R
- added R51, R52: 5.1k, Resistor_SMD:R_0805_2012Metric, symbol zl80:R
- C27, C28, C32, C33, C34, C5: footprint Capacitor_THT:C_Disc_D5.0mm_W2.5mm_P5.00mm -> Capacitor_SMD:C_0805_2012Metric
- J6: value PS/2 keyboard -> PS/2 keyboard (panel socket); footprint (none) -> Connector_PinHeader_2.54mm:PinHeader_1x04_P2.54mm_Vertical; symbol zl80:MiniDIN6_PS2 -> zl80:PS2_Header
- R12, R13, R14: footprint Resistor_THT:R_Axial_DIN0207_L6.3mm_D2.5mm_P10.16mm_Horizontal -> Resistor_SMD:R_0805_2012Metric
- U21: footprint Package_DIP:DIP-40_W15.24mm -> Package_DIP:DIP-40_W15.24mm_Socket
- U22: value ATmega328P: PS/2 to key matrix -> ATmega328P-AU: PS/2 to key matrix; footprint Package_DIP:DIP-28_W7.62mm -> Package_QFP:TQFP-32_7x7mm_P0.8mm; symbol zl80:ATmega328P -> zl80:ATmega328P-AU
- U23: value UM245R USB FIFO module -> FT245RL USB FIFO; footprint Package_DIP:DIP-24_W15.24mm -> Package_SO:SSOP-28_5.3x10.2mm_P0.65mm; symbol zl80:UM245R -> zl80:FT245RL
- U27, U28: footprint Package_DIP:DIP-14_W7.62mm -> Package_SO:SOIC-14_3.9x8.7mm_P1.27mm
Connections:
- net +5V: now also J6.1 (+5V (DIN 4)), U22.18 (AVCC), U22.4 (VCC), U22.6 (VCC), U23.20 (VCC), U23.4 (VCCIO), C37.1, C38.1, R50.1; no longer J6.4 (+5V), U22.20 (AVCC), U22.7 (VCC), U23.15 (VCC), U23.21 (VCC)
- net D3: now also U23.11 (D3); no longer U23.10 (DB3)
- net D5: now also U23.9 (D5); no longer U23.8 (DB5)
- net D6: now also U23.10 (D6); no longer U23.9 (DB6)
- net GND: now also J6.4 (GND (DIN 3, shell)), U22.21 (GND), U22.3 (GND), U22.5 (GND), U23.18 (GND), U23.21 (GND), U23.25 (AGND), U23.26 (TEST), C36.2, C37.2, C38.2, C39.2, J10.A1 (GND), J10.A12 (GND), J10.B1 (GND), J10.B12 (GND), R49.2, R51.2, R52.2; no longer J6.3 (GND), J6.SH (Shield), U22.22 (GND), U22.8 (GND), U23.24 (GND)
- net KB_AREF: now also U22.20 (AREF); no longer U22.21 (AREF)
- net KB_MISO: now also U22.16 (PB4/MISO); no longer U22.18 (PB4/MISO)
- net KB_MOSI: now also U22.15 (PB3/MOSI); no longer U22.17 (PB3/MOSI)
- net KB_RST: now also U22.29 (PC6/~{RESET}); no longer U22.1 (PC6/~{RESET})
- net KB_SCK: now also U22.17 (PB5/SCK); no longer U22.19 (PB5/SCK)
- net KCOL0: now also U22.30 (PD0); no longer U22.2 (PD0)
- net KCOL1: now also U22.31 (PD1); no longer U22.3 (PD1)
- net KCOL2: now also U22.32 (PD2); no longer U22.4 (PD2)
- net KCOL3: now also U22.1 (PD3); no longer U22.5 (PD3)
- net KCOL4: now also U22.2 (PD4); no longer U22.6 (PD4)
- net KCOL5: now also U22.9 (PD5); no longer U22.11 (PD5)
- net KCOL6: now also U22.10 (PD6); no longer U22.12 (PD6)
- net KCOL7: now also U22.11 (PD7); no longer U22.13 (PD7)
- net PS2_CLK: now also J6.2 (Clock (DIN 5)), U22.12 (PB0); no longer J6.5 (Clock), U22.14 (PB0)
- net PS2_DATA: now also J6.3 (Data (DIN 1)), U22.13 (PB1); no longer J6.1 (Data), U22.15 (PB1)
- net USBWR: now also U23.14 (WR); no longer U23.18 (WR)
- net USB_RST: now also U23.19 (~{RESET}), R48.2, R49.1; no longer U23.17 (PU1), U23.20 (RST#)
- net USB_VBUS: now also J10.A4 (VBUS), J10.A9 (VBUS), J10.B4 (VBUS), J10.B9 (VBUS), R48.1; no longer U23.14 (USB (5V out)), U23.16 (PU2)
- net ~{USBRD}: now also U23.13 (~{RD}); no longer U23.12 (RD#)
- new net USB_3V3: C36.1, U23.17 (3V3OUT)
- new net USB_CC1: J10.A5 (CC1), R51.1
- new net USB_CC2: J10.B5 (CC2), R52.1
- new net USB_DM: J10.A7 (D-), J10.B7 (D-), U23.16 (USBDM)
- new net USB_DP: J10.A6 (D+), J10.B6 (D+), U23.15 (USBDP)
- new net USB_PWREN: R50.2, U23.12 (~{PWREN})
- new net USB_SHIELD: C39.1, J10.S1 (SHIELD)
- no-connect marks 13 -> 15
Other:
- moved on the sheet: C27, C28, C32, C33, C34, C5, J7, R12, R13, R14
