File: hardware/kicad/power_tv.kicad_sch (KiCad schematic)
At the start: 14 parts, among them J1 12 V DC in, J2 SCART, J3 RGB board (later), SW1 Reset, U13 DS1813-5 reset, U14 R-78E5.0-1.0 (or 7805)

Commit message: Add the routed 4-layer PCB and move the board to SMD parts
Schematic:
- Z80, TMS9918A, AY-3-8910 and 82C55 stay DIP-40 in sockets (the
  chips in hand), the SST39SF040 flash is a socketed DIP-32 so it can
  be programmed; everything else is surface mount: AS6C4008 SOP-32,
  AS6C62256 SOP-28 VRAM, logic in SOIC, ATmega328P-AU TQFP-32, 0805.
- The UM245R module becomes an FT245RL (SSOP-28) with a USB-C socket
  (GCT USB4105), wired as FTDI's self-powered figure 6.2.
- 74HC670 instead of the 74HCT670, no longer made in SOIC; all its
  inputs come from CMOS outputs.
- MMBT4401 video transistor with SOT-23 pins 1 B, 2 E, 3 C; the TO-92
  pin numbers used before were wrong.
- SCART and PS/2 go to headers for short cables (no KiCad footprints;
  smaller board). DB9s, USB-C and the 12 V jack stay on the board.
- Pin tables checked against the manufacturers' datasheets;
  check_footprints.py confirms every symbol pin has a pad.

PCB (gen_pcb.py, KiCad 9 Python):
- 138 x 105 mm, 4 layers: tracks on F.Cu, In2.Cu and B.Cu, In1.Cu an
  unbroken GND plane, +5V as 0.4 mm tracks plus a fill on In2.Cu.
- Connectors on the top edge, the DIP sockets in one row, each
  group's SMD parts packed beside and below its socket with each
  chip's 100 nF next to it. One-sided SMD assembly.
- Routed with Freerouting 2.5.0. The DSN is adjusted so only GND may
  use In1.Cu and the boundary is inset by the edge clearance.
- KiCad DRC with schematic parity: 0 violations, 0 unconnected pads,
  0 footprint errors. Only silkscreen warnings remain. ERC 0.

Not built or tested.

Co-Authored-By: Claude Opus 5.5 <noreply@anthropic.com>
Parts:
- removed J3: RGB board (later), Connector_PinHeader_2.54mm:PinHeader_1x07_P2.54mm_Vertical, symbol zl80:RGB_Header
- C3, C4: footprint Capacitor_THT:CP_Radial_D6.3mm_P2.50mm -> Capacitor_SMD:CP_Elec_6.3x7.7
- D1: value 1N5819 -> 1N5819HW; footprint Diode_THT:D_DO-41_SOD81_P10.16mm_Horizontal -> Diode_SMD:D_SOD-123
- D2: footprint LED_THT:LED_D3.0mm -> LED_SMD:LED_0805_2012Metric
- J2: value SCART -> TV: cable to a SCART plug; footprint (none) -> Connector_PinHeader_2.54mm:PinHeader_2x05_P2.54mm_Vertical; symbol zl80:SCART -> zl80:TV_Header
- R15, R28, R29, R32: footprint Resistor_THT:R_Axial_DIN0207_L6.3mm_D2.5mm_P10.16mm_Horizontal -> Resistor_SMD:R_0805_2012Metric
- SW1: footprint Button_Switch_THT:SW_PUSH_6mm -> Button_Switch_SMD:SW_SPST_B3U-1000P
- U13: footprint Package_TO_SOT_THT:TO-92_Inline -> Package_TO_SOT_SMD:SOT-23-3
- U14: footprint Package_TO_SOT_THT:TO-220-3_Vertical -> Converter_DCDC:Converter_DCDC_RECOM_R-78E-0.5_THT
Connections:
- net RGB_B is gone; now on net BLANK: J2.7 (Blanking (SCART 16))
- net +5V: now also J2.10 (+5V)
- net AUD_L: now also J2.3 (Audio L (SCART 6)); no longer J2.6 (Audio L in)
- net AUD_R: now also J2.4 (Audio R (SCART 2)); no longer J2.2 (Audio R in)
- net BLANK: no longer J2.16 (Blanking)
- net EXTVDP: now also J2.9 (EXTVDP)
- net GND: now also J2.2 (GND (SCART 17)), J2.8 (GND (SCART 18, 21)); no longer J2.13 (Red GND), J2.14 (Data GND), J2.17 (Video GND), J2.18 (Blanking GND), J2.21 (Shield), J2.4 (Audio GND), J2.9 (Green GND)
- net SCART_FS: now also J2.6 (12V switch (SCART 8)); no longer J2.8 (Function switch)
- net VID_OUT: now also J2.1 (Video (SCART 20)); no longer J2.20 (Video in)
- removed net RGB_G: J2.11 (Green)
- removed net RGB_R: J2.15 (Red)
- no-connect marks 5 -> 0
