File: hardware/kicad/sound.kicad_sch (KiCad schematic)
At the start: 25 parts, among them J4 Joystick 1 (Atari / Sega), J5 Joystick 2 (Atari / Sega), U12 74HCT02 AY bus control, USB WR, U18 AY-3-8910, U19 74HCT157 joystick directions, U20 74HCT157 joystick buttons

Commit message: Add the routed 4-layer PCB and move the board to SMD parts
Schematic:
- Z80, TMS9918A, AY-3-8910 and 82C55 stay DIP-40 in sockets (the
  chips in hand), the SST39SF040 flash is a socketed DIP-32 so it can
  be programmed; everything else is surface mount: AS6C4008 SOP-32,
  AS6C62256 SOP-28 VRAM, logic in SOIC, ATmega328P-AU TQFP-32, 0805.
- The UM245R module becomes an FT245RL (SSOP-28) with a USB-C socket
  (GCT USB4105), wired as FTDI's self-powered figure 6.2.
- 74HC670 instead of the 74HCT670, no longer made in SOIC; all its
  inputs come from CMOS outputs.
- MMBT4401 video transistor with SOT-23 pins 1 B, 2 E, 3 C; the TO-92
  pin numbers used before were wrong.
- SCART and PS/2 go to headers for short cables (no KiCad footprints;
  smaller board). DB9s, USB-C and the 12 V jack stay on the board.
- Pin tables checked against the manufacturers' datasheets;
  check_footprints.py confirms every symbol pin has a pad.

PCB (gen_pcb.py, KiCad 9 Python):
- 138 x 105 mm, 4 layers: tracks on F.Cu, In2.Cu and B.Cu, In1.Cu an
  unbroken GND plane, +5V as 0.4 mm tracks plus a fill on In2.Cu.
- Connectors on the top edge, the DIP sockets in one row, each
  group's SMD parts packed beside and below its socket with each
  chip's 100 nF next to it. One-sided SMD assembly.
- Routed with Freerouting 2.5.0. The DSN is adjusted so only GND may
  use In1.Cu and the boundary is inset by the edge clearance.
- KiCad DRC with schematic parity: 0 violations, 0 unconnected pads,
  0 footprint errors. Only silkscreen warnings remain. ERC 0.

Not built or tested.

Co-Authored-By: Claude Opus 5.5 <noreply@anthropic.com>
Parts:
- removed RN1, RN2: 10k x 8, Resistor_THT:R_Array_SIP9, symbol zl80:R_Network08
- added R33, R34, R35, R36, R37, R38, R39, R40, R41, R42, R43, R44, R45, R46, R47: 10k, Resistor_SMD:R_0805_2012Metric, symbol zl80:R
- C1, C2: footprint Capacitor_THT:CP_Radial_D6.3mm_P2.50mm -> Capacitor_SMD:C_0805_2012Metric; symbol zl80:C_Polarized -> zl80:C
- C23, C24, C25, C26: footprint Capacitor_THT:C_Disc_D5.0mm_W2.5mm_P5.00mm -> Capacitor_SMD:C_0805_2012Metric
- J4, J5: footprint (none) -> Connector_Dsub:DSUB-9_Male_Horizontal_P2.77x2.84mm_EdgePinOffset7.70mm_Housed_MountingHolesOffset9.12mm
- R16, R17, R18, R19, R20, R21, R22, R23, R24, R30, R31: footprint Resistor_THT:R_Axial_DIN0207_L6.3mm_D2.5mm_P10.16mm_Horizontal -> Resistor_SMD:R_0805_2012Metric
- U12: footprint Package_DIP:DIP-14_W7.62mm -> Package_SO:SOIC-14_3.9x8.7mm_P1.27mm
- U18: footprint Package_DIP:DIP-40_W15.24mm -> Package_DIP:DIP-40_W15.24mm_Socket
- U19, U20: footprint Package_DIP:DIP-16_W7.62mm -> Package_SO:SOIC-16_3.9x9.9mm_P1.27mm
Connections:
- net +5V: now also R33.1, R34.1, R35.1, R36.1, R37.1, R38.1, R39.1, R40.1, R41.1, R42.1, R43.1, R44.1, R45.1, R46.1, R47.1
- net GND: now also J4.0 (Shield), J5.0 (Shield); no longer J4.SH (Shield), J5.SH (Shield)
- net IOA6: now also R45.2
- net IOA7: now also R46.2
- net J1_B1: now also R37.2
- net J1_B2: now also R38.2
- net J1_DOWN: now also R34.2
- net J1_LEFT: now also R35.2
- net J1_RIGHT: now also R36.2
- net J1_UP: now also R33.2
- net J2_B1: now also R43.2
- net J2_B2: now also R44.2
- net J2_DOWN: now also R40.2
- net J2_LEFT: now also R41.2
- net J2_RIGHT: now also R42.2
- net J2_UP: now also R39.2
- net JOYSEL: now also R47.2
- no-connect marks 15 -> 14
Other:
- moved on the sheet: C23, C24, C25, C26, R30, R31
