File: hardware/kicad/video.kicad_sch (KiCad schematic)
At the start: 22 parts, among them Q1 2N4401 video buffer, U15 TMS9918A, U16 62256 VRAM (16 KB used), U17 74HCT574 VRAM row latch, U24 74HCT574 VRAM column latch, U25 74HCT574 VRAM write data, U26 74HCT04 VRAM strobes, Y1 10.738635 MHz

Commit message: Add the routed 4-layer PCB and move the board to SMD parts
Schematic:
- Z80, TMS9918A, AY-3-8910 and 82C55 stay DIP-40 in sockets (the
  chips in hand), the SST39SF040 flash is a socketed DIP-32 so it can
  be programmed; everything else is surface mount: AS6C4008 SOP-32,
  AS6C62256 SOP-28 VRAM, logic in SOIC, ATmega328P-AU TQFP-32, 0805.
- The UM245R module becomes an FT245RL (SSOP-28) with a USB-C socket
  (GCT USB4105), wired as FTDI's self-powered figure 6.2.
- 74HC670 instead of the 74HCT670, no longer made in SOIC; all its
  inputs come from CMOS outputs.
- MMBT4401 video transistor with SOT-23 pins 1 B, 2 E, 3 C; the TO-92
  pin numbers used before were wrong.
- SCART and PS/2 go to headers for short cables (no KiCad footprints;
  smaller board). DB9s, USB-C and the 12 V jack stay on the board.
- Pin tables checked against the manufacturers' datasheets;
  check_footprints.py confirms every symbol pin has a pad.

PCB (gen_pcb.py, KiCad 9 Python):
- 138 x 105 mm, 4 layers: tracks on F.Cu, In2.Cu and B.Cu, In1.Cu an
  unbroken GND plane, +5V as 0.4 mm tracks plus a fill on In2.Cu.
- Connectors on the top edge, the DIP sockets in one row, each
  group's SMD parts packed beside and below its socket with each
  chip's 100 nF next to it. One-sided SMD assembly.
- Routed with Freerouting 2.5.0. The DSN is adjusted so only GND may
  use In1.Cu and the boundary is inset by the edge clearance.
- KiCad DRC with schematic parity: 0 violations, 0 unconnected pads,
  0 footprint errors. Only silkscreen warnings remain. ERC 0.

Not built or tested.

Co-Authored-By: Claude Opus 5.5 <noreply@anthropic.com>
Parts:
- C17, C18, C19, C20, C21, C22, C29, C30, C31: footprint Capacitor_THT:C_Disc_D5.0mm_W2.5mm_P5.00mm -> Capacitor_SMD:C_0805_2012Metric
- D3: value BAT85 -> 1N5819HW; footprint Diode_THT:D_DO-41_SOD81_P10.16mm_Horizontal -> Diode_SMD:D_SOD-123
- FB1: footprint Inductor_THT:L_Axial_L5.3mm_D2.2mm_P7.62mm_Horizontal_Vishay_IM-1 -> Inductor_SMD:L_0805_2012Metric
- Q1: value 2N4401 video buffer -> MMBT4401 video buffer; footprint Package_TO_SOT_THT:TO-92_Inline -> Package_TO_SOT_SMD:SOT-23-3; symbol zl80:NPN_BCE -> zl80:NPN_SOT23
- R25, R26, R27: footprint Resistor_THT:R_Axial_DIN0207_L6.3mm_D2.5mm_P10.16mm_Horizontal -> Resistor_SMD:R_0805_2012Metric
- U15: footprint Package_DIP:DIP-40_W15.24mm -> Package_DIP:DIP-40_W15.24mm_Socket
- U16: footprint Package_DIP:DIP-28_W15.24mm -> Package_SO:SOP-28_8.4x18.16mm_P1.27mm
- U17, U24, U25: footprint Package_DIP:DIP-20_W7.62mm -> Package_SO:SOIC-20W_7.5x12.8mm_P1.27mm
- U26: footprint Package_DIP:DIP-14_W7.62mm -> Package_SO:SOIC-14_3.9x8.7mm_P1.27mm
- Y1: footprint Crystal:Crystal_HC49-4H_Vertical -> Crystal:Crystal_SMD_HC49-SD
Connections:
- net VID_B: now also Q1.1 (B); no longer Q1.2 (B)
- net VID_C: now also Q1.3 (C); no longer Q1.1 (C)
- net VID_OUT: now also Q1.2 (E); no longer Q1.3 (E)

Commit message: Add schematic, PCB and 3D pictures to the READMEs
hardware/images holds the six schematic pages and the copper layers
as SVG (kicad-cli sch/pcb export svg) and three 3D renders as PNG
(kicad-cli pcb render: top, bottom, angled). The main README shows
the 3D views and links every schematic page and layer; the KiCad
README shows the angled view and says how to export them again.

The video page is now "Video, TMS9918A and VRAM": the colon in its
old name made an invalid Windows file name when exported. ERC and
the PCB schematic parity check are still clean.

Co-Authored-By: Claude Opus 5.5 <noreply@anthropic.com>
Other:
- title: Video: TMS9918A and VRAM -> Video, TMS9918A and VRAM
Changed lines of the file:
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@@
 (kicad_sch (version 20230121) (generator eeschema)
   (paper "A2")
-  (title_block (title "Video: TMS9918A and VRAM") (date "2026-10-27") (rev "0.3")
+  (title_block (title "Video, TMS9918A and VRAM") (date "2026-10-27") (rev "0.3")
     (comment 1 "Z80 3.58 MHz, TMS9918A + 16 KB SRAM VRAM, AY-3-8910, 512 KB flash + 512 KB SRAM, 82C55 + PS/2, FT245RL USB-C")
     (comment 2 "Design only: not built or tested")
